File: Kicad/Atmega_328_breakout.sch (KiCad schematic (older format))
At the start: 71 parts, among them J1 Jack-DC, J10 Conn_01x06, J11 1x2, J12 1x2, J13 1x2, J14 1x2, J15 1x2, J16 1x2, J17 1x2, J18 1x2, J19 Power_connector, J2 1x2, J20 ADC_Connector, J21 PORB++_connector, J22 PORD_connector, J23 Conn_01x01, J24 Device_Connector, J25 Pin out, J26 Com_header, J27 Power terminal, J28 USB, J3 1x2, J4 1x2, J5 1x2, J6 1x2, J7 1x2, J8 1x2, J9 1x2, Q1 PMOS, SW1 SW_Push, SW2 SW_Push, U1 NCP1117-5, U2 L7805, U3 TL071, U4 ATMEGA328P-AU, U5 MCP1700-33, U6 MCP2221, Y1 Crystal

Commit message: last commit before merge
Parts:
- U4: LCSC (none) -> C132230
Connections:
- wire segments 320 -> 317
Other:
- note added: "Normal Pin headers"
- note removed: "Arduino Shield and normal Pin headers"
- moved on the sheet: C1, C10, C3, C4, J10, J21, J22, J23, J24, SHIELD1, U4

Commit message: double checked files
Parts:
- C1, C10, C11, C12, C13, C14, C2, C3, C4, C5, C6, C7, C8, C9: symbol Atmega_328_breakout-rescue:C_Small -> Atmega_328_breakout-rescue:C_Small-Atmega_328_breakout-rescue
- D1: symbol Atmega_328_breakout-rescue:D_Schottky -> Atmega_328_breakout-rescue:D_Schottky-Atmega_328_breakout-rescue
- D2: symbol Atmega_328_breakout-rescue:D_Zener -> Atmega_328_breakout-rescue:D_Zener-Atmega_328_breakout-rescue
- D3, D4: symbol Atmega_328_breakout-rescue:LED -> Atmega_328_breakout-rescue:LED-Atmega_328_breakout-rescue
- F1: symbol Atmega_328_breakout-rescue:Polyfuse -> Atmega_328_breakout-rescue:Polyfuse-Atmega_328_breakout-rescue
- ISP1: symbol Atmega_328_breakout-rescue:AVR-ISP-6 -> Atmega_328_breakout-rescue:AVR-ISP-6-Atmega_328_breakout-rescue
- J1: symbol Atmega_328_breakout-rescue:Jack-DC -> Atmega_328_breakout-rescue:Jack-DC-Atmega_328_breakout-rescue
- J10: symbol Atmega_328_breakout-rescue:Conn_01x06 -> Atmega_328_breakout-rescue:Conn_01x06-Atmega_328_breakout-rescue
- J11, J12, J13, J14, J15, J16, J17, J18, J2, J3, J4, J5, J6, J7, J8, J9: symbol Atmega_328_breakout-rescue:Conn_01x02_Female -> Atmega_328_breakout-rescue:Conn_01x02_Female-Atmega_328_breakout-rescue
- J19: symbol Atmega_328_breakout-rescue:Conn_01x06_Female -> Atmega_328_breakout-rescue:Conn_01x06_Female-Atmega_328_breakout-rescue
- J20, J21, J22: symbol Atmega_328_breakout-rescue:Conn_01x08_Female -> Atmega_328_breakout-rescue:Conn_01x08_Female-Atmega_328_breakout-rescue
- J23: symbol Atmega_328_breakout-rescue:Conn_01x01 -> Atmega_328_breakout-rescue:Conn_01x01-Atmega_328_breakout-rescue
- J24, J25: symbol Atmega_328_breakout-rescue:Conn_01x03_Female -> Atmega_328_breakout-rescue:Conn_01x03_Female-Atmega_328_breakout-rescue
- J26: symbol Atmega_328_breakout-rescue:Conn_02x05_Odd_Even -> Atmega_328_breakout-rescue:Conn_02x05_Odd_Even-Atmega_328_breakout-rescue
- J27: symbol Atmega_328_breakout-rescue:Conn_01x09 -> Atmega_328_breakout-rescue:Conn_01x09-Atmega_328_breakout-rescue
- J28: symbol Atmega_328_breakout-rescue:USB_OTG -> Atmega_328_breakout-rescue:USB_OTG-Atmega_328_breakout-rescue
- L1, L2, L3: symbol Atmega_328_breakout-rescue:Ferrite_Bead_Small -> Atmega_328_breakout-rescue:Ferrite_Bead_Small-Atmega_328_breakout-rescue
- Q1: symbol Atmega_328_breakout-rescue:Q_PMOS_SGD -> Atmega_328_breakout-rescue:Q_PMOS_SGD-Atmega_328_breakout-rescue
- R1, R2, R3, R4, R5, R6, R7, R8, R9: symbol Atmega_328_breakout-rescue:R -> Atmega_328_breakout-rescue:R-Atmega_328_breakout-rescue
- SHIELD1: symbol Atmega_328_breakout-rescue:ATMEL_SHIELD -> Atmega_328_breakout-rescue:ATMEL_SHIELD-Atmega_328_breakout-rescue
- SW1, SW2: symbol Atmega_328_breakout-rescue:SW_Push -> Atmega_328_breakout-rescue:SW_Push-Atmega_328_breakout-rescue
- U1: symbol Atmega_328_breakout-rescue:NCP1117-5.0_SOT223 -> Atmega_328_breakout-rescue:NCP1117-5.0_SOT223-Atmega_328_breakout-rescue
- U2: symbol Atmega_328_breakout-rescue:L7805 -> Atmega_328_breakout-rescue:L7805-Atmega_328_breakout-rescue
- U4: symbol Atmega_328_breakout-rescue:ATMEGA328P-AU -> Atmega_328_breakout-rescue:ATMEGA328P-AU-Atmega_328_breakout-rescue
- U6: symbol Atmega_328_breakout-rescue:MCP2221 -> Atmega_328_breakout-rescue:MCP2221-Atmega_328_breakout-rescue
- Y1: symbol Atmega_328_breakout-rescue:Crystal -> Atmega_328_breakout-rescue:Crystal-Atmega_328_breakout-rescue

Commit message: copied edited files
Parts:
- C1, C10, C11, C12, C13, C14, C2, C3, C4, C5, C6, C7, C8, C9: symbol Atmega_328_breakout-rescue:C_Small-Atmega_328_breakout-rescue -> Atmega_328_breakout-rescue:C_Small
- D1: symbol Atmega_328_breakout-rescue:D_Schottky-Atmega_328_breakout-rescue -> Atmega_328_breakout-rescue:D_Schottky
- D2: symbol Atmega_328_breakout-rescue:D_Zener-Atmega_328_breakout-rescue -> Atmega_328_breakout-rescue:D_Zener
- D3, D4: symbol Atmega_328_breakout-rescue:LED-Atmega_328_breakout-rescue -> Atmega_328_breakout-rescue:LED
- F1: symbol Atmega_328_breakout-rescue:Polyfuse-Atmega_328_breakout-rescue -> Atmega_328_breakout-rescue:Polyfuse
- ISP1: symbol Atmega_328_breakout-rescue:AVR-ISP-6-Atmega_328_breakout-rescue -> Atmega_328_breakout-rescue:AVR-ISP-6
- J1: symbol Atmega_328_breakout-rescue:Jack-DC-Atmega_328_breakout-rescue -> Atmega_328_breakout-rescue:Jack-DC
- J10: symbol Atmega_328_breakout-rescue:Conn_01x06-Atmega_328_breakout-rescue -> Atmega_328_breakout-rescue:Conn_01x06
- J11, J12, J13, J14, J15, J16, J17, J18, J2, J3, J4, J5, J6, J7, J8, J9: symbol Atmega_328_breakout-rescue:Conn_01x02_Female-Atmega_328_breakout-rescue -> Atmega_328_breakout-rescue:Conn_01x02_Female
- J19: symbol Atmega_328_breakout-rescue:Conn_01x06_Female-Atmega_328_breakout-rescue -> Atmega_328_breakout-rescue:Conn_01x06_Female
- J20, J21, J22: symbol Atmega_328_breakout-rescue:Conn_01x08_Female-Atmega_328_breakout-rescue -> Atmega_328_breakout-rescue:Conn_01x08_Female
- J23: symbol Atmega_328_breakout-rescue:Conn_01x01-Atmega_328_breakout-rescue -> Atmega_328_breakout-rescue:Conn_01x01
- J24, J25: symbol Atmega_328_breakout-rescue:Conn_01x03_Female-Atmega_328_breakout-rescue -> Atmega_328_breakout-rescue:Conn_01x03_Female
- J26: symbol Atmega_328_breakout-rescue:Conn_02x05_Odd_Even-Atmega_328_breakout-rescue -> Atmega_328_breakout-rescue:Conn_02x05_Odd_Even
- J27: symbol Atmega_328_breakout-rescue:Conn_01x09-Atmega_328_breakout-rescue -> Atmega_328_breakout-rescue:Conn_01x09
- J28: symbol Atmega_328_breakout-rescue:USB_OTG-Atmega_328_breakout-rescue -> Atmega_328_breakout-rescue:USB_OTG
- L1, L2, L3: symbol Atmega_328_breakout-rescue:Ferrite_Bead_Small-Atmega_328_breakout-rescue -> Atmega_328_breakout-rescue:Ferrite_Bead_Small
- Q1: symbol Atmega_328_breakout-rescue:Q_PMOS_SGD-Atmega_328_breakout-rescue -> Atmega_328_breakout-rescue:Q_PMOS_SGD
- R1, R2, R3, R4, R5, R6, R7, R8, R9: symbol Atmega_328_breakout-rescue:R-Atmega_328_breakout-rescue -> Atmega_328_breakout-rescue:R
- SHIELD1: symbol Atmega_328_breakout-rescue:ATMEL_SHIELD-Atmega_328_breakout-rescue -> Atmega_328_breakout-rescue:ATMEL_SHIELD
- SW1, SW2: symbol Atmega_328_breakout-rescue:SW_Push-Atmega_328_breakout-rescue -> Atmega_328_breakout-rescue:SW_Push
- U1: symbol Atmega_328_breakout-rescue:NCP1117-5.0_SOT223-Atmega_328_breakout-rescue -> Atmega_328_breakout-rescue:NCP1117-5.0_SOT223
- U2: symbol Atmega_328_breakout-rescue:L7805-Atmega_328_breakout-rescue -> Atmega_328_breakout-rescue:L7805
- U4: symbol Atmega_328_breakout-rescue:ATMEGA328P-AU-Atmega_328_breakout-rescue -> Atmega_328_breakout-rescue:ATMEGA328P-AU
- U6: symbol Atmega_328_breakout-rescue:MCP2221-Atmega_328_breakout-rescue -> Atmega_328_breakout-rescue:MCP2221
- Y1: symbol Atmega_328_breakout-rescue:Crystal-Atmega_328_breakout-rescue -> Atmega_328_breakout-rescue:Crystal
