File: Kicad/Atmega_328_breakout.sch (KiCad schematic (older format))
At the start: 71 parts, among them J1 Jack-DC, J10 Conn_01x06, J11 01x03, J12 01x03, J13 01x03, J14 01x03, J15 01x03, J16 01x03, J17 01x03, J18 01x03, J19 Power_connector, J2 01x03, J20 ADC_Connector, J21 PORB++_connector, J22 PORD_connector, J23 Conn_01x01, J24 Device_Connector, J25 Pin out, J26 Com_header, J27 Power terminal, J28 USB, J3 01x03, J4 01x03, J5 01x03, J6 01x03, J7 01x03, J8 01x03, J9 01x03, Q1 PMOS, SW1 SW_Push, SW2 SW_Push, U1 NCP1117-5, U2 L7805, U3 LM358, U4 ATMEGA328P-AU, U5 MCP1700-33, U6 MCP2221, Y1 Crystal_GND24

Commit message: started adding new parts
Parts:
- removed U6: MCP2221, Package_SO:TSSOP-14_4.4x5mm_P0.65mm, symbol Atmega_328_breakout-rescue:MCP2221
- added C15: 100n, Capacitor_SMD:C_0603_1608Metric_Pad1.08x0.95mm_HandSolder, symbol Atmega_328_breakout-rescue:C_Small
- added C16, C17: 33p, Capacitor_SMD:C_0603_1608Metric_Pad1.08x0.95mm_HandSolder, symbol Atmega_328_breakout-rescue:C_Small
- added U6: CH340G, Package_SO:SOIC-16_3.9x9.9mm_P1.27mm, symbol Interface_USB:CH340G
- added Y2: Crystal_GND24_12MHz, Crystal:Crystal_SMD_3225-4Pin_3.2x2.5mm, symbol Device:Crystal_GND24
- Y1: value Crystal_GND24 -> Crystal_GND24_16MHz
Connections:
- net GND: now also C15.2, C16.1, C17.1, U6.1 (GND), Y2.2, Y2.4
- net PD0(RX): now also U6.2 (TXD)
- net PD1(TX): now also U6.3 (RXD)
- net VCC: now also U6.16 (VCC)
- net ~RESET: now also U6.14 (~RTS)
- net at J28.2 (D-): now also U6.6 (UD-)
- net at J28.3 (D+): now also U6.5 (UD+)
- new net: C15.1, U6.4 (V3)
- new net: C17.2, U6.7 (XI), Y2.3
- new net: C16.2, U6.8 (XO), Y2.1
Other:
- moved on the sheet: C14, J28
