File: Kicad/Atmega_328_breakout.sch (KiCad schematic (older format))
At the start: 70 parts, among them J1 Jack-DC, J10 Conn_01x06, J11 1x2, J12 1x2, J13 1x2, J14 1x2, J15 1x2, J16 1x2, J17 1x2, J18 1x2, J19 Power_connector, J2 1x2, J20 ADC_Connector, J21 PORB++_connector, J22 PORD_connector, J23 Conn_01x01, J24 Device_Connector, J25 Pin out, J26 Com_header, J27 Power terminal, J28 USB, J3 1x2, J4 1x2, J5 1x2, J6 1x2, J7 1x2, J8 1x2, J9 1x2, Q1 PMOS, SW1 SW_Push, SW2 SW_Push, U1 NCP1117-5, U2 L7805, U3 TL071, U4 ATMEGA328P-AU, U5 MCP1700-33, U6 MCP2221, Y1 Crystal

Commit message: All parts added and part number
Parts:
- removed J11, J12, J13, J14, J15, J16, J17, J18, J2, J3, J4, J5, J6, J7, J8, J9: 1x2, jorgen:Pin_Header_Straight_1x02_Pitch2.54mm, symbol Atmega_328_breakout-rescue:Conn_01x02_Female
- removed Y1: Crystal, Crystal:Crystal_HC49-U_Vertical, symbol Atmega_328_breakout-rescue:Crystal
- added J11, J12, J13, J14, J15, J16, J17, J18, J2, J3, J4, J5, J6, J7, J8, J9: 01x03, jorgen:conn_01x03_square, symbol Connector:Conn_01x03_Male
- added Y1: Crystal_GND24, Crystal:Crystal_SMD_3225-4Pin_3.2x2.5mm, symbol Device:Crystal_GND24
- D2: footprint Diode_SMD:D_0603_1608Metric -> Diode_SMD:D_SC-80_HandSoldering; LCSC (none) -> C8062
- F1: LCSC (none) -> C66453
- J10: footprint Connector_PinHeader_2.54mm:PinHeader_2x03_P2.54mm_Vertical -> Connector_PinSocket_2.54mm:PinSocket_2x03_P2.54mm_Vertical
- J19: footprint Connector_PinHeader_2.54mm:PinHeader_1x06_P2.54mm_Vertical -> Connector_PinSocket_2.54mm:PinSocket_1x06_P2.54mm_Vertical
- J20, J21, J22: footprint Connector_PinHeader_2.54mm:PinHeader_1x08_P2.54mm_Vertical -> Connector_PinSocket_2.54mm:PinSocket_1x08_P2.54mm_Vertical
- SW1, SW2: LCSC (none) -> C318887
Connections:
- wire segments 312 -> 331

Commit message: before switching
Parts:
- R1: value 10kR -> 5k
- R2: value 20k -> 30k
- U1: footprint Package_TO_SOT_SMD:SOT-23 -> Package_TO_SOT_SMD:SOT-223-3_TabPin2; LCSC (none) -> C17314
Other:
- moved on the sheet: C12
Changed lines of the file:
@@
 L Atmega_328_breakout-rescue:C_Small C12
 U 1 1 5A7309D9
-P 4150 1550
-F 0 "C12" H 4160 1620 50  0000 L CNN
-F 1 "22p" H 4160 1470 50  0000 L CNN
-F 2 "Capacitor_SMD:C_0603_1608Metric_Pad1.08x0.95mm_HandSolder" H 4150 1550 50  0001 C CNN
-F 3 "" H 4150 1550 50  0001 C CNN
-F 4 "C1653" H 4150 1550 50  0001 C CNN "LCSC"
-	1    4150 1550
+P 4050 1550
+F 0 "C12" H 4060 1620 50  0000 L CNN
+F 1 "22p" H 4060 1470 50  0000 L CNN
+F 2 "Capacitor_SMD:C_0603_1608Metric_Pad1.08x0.95mm_HandSolder" H 4050 1550 50  0001 C CNN
+F 3 "" H 4050 1550 50  0001 C CNN
+F 4 "C1653" H 4050 1550 50  0001 C CNN "LCSC"
+	1    4050 1550
 	-1   0    0    1
 $EndComp
@@
 AGND
 Wire Wire Line
-	1450 7800 1450 7875
-Wire Wire Line
-	3100 8275 2450 8275
-Wire Wire Line
-	1850 8175 1450 8175
-Wire Wire Line
 	1700 8375 1850 8375
 NoConn ~ 1000 6650
@@
 F 0 "U1" H 1350 9975 50  0000 C CNN
 F 1 "NCP1117-5" H 1500 9975 50  0000 L CNN
-F 2 "Package_TO_SOT_SMD:SOT-23" H 1500 10050 50  0001 C CNN
+F 2 "Package_TO_SOT_SMD:SOT-223-3_TabPin2" H 1500 10050 50  0001 C CNN
 F 3 "" H 1600 9600 50  0001 C CNN
-F 4 "" H 1500 9850 50  0001 C CNN "LCSC"
+F 4 "C17314" H 1500 9850 50  0001 C CNN "LCSC"
 	1    1500 9850
 	1    0    0    -1
@@
 	0    -1   -1   0
 $EndComp
-NoConn ~ 2150 8575
-NoConn ~ 2250 8575
 $Comp
 L Atmega_328_breakout-rescue:+5V #PWR08
@@
 $EndComp
 $Comp
-L power:GND #PWR06
-U 1 1 5A7493FE
-P 1450 8475
-F 0 "#PWR06" H 1450 8225 50  0001 C CNN
-F 1 "GND" H 1450 8325 50  0000 C CNN
-F 2 "" H 1450 8475 50  0001 C CNN
-F 3 "" H 1450 8475 50  0001 C CNN
-	1    1450 8475
-	1    0    0    -1
-$EndComp
-$Comp
-L Atmega_328_breakout-rescue:R R1
-U 1 1 5A749034
-P 1450 8025
-F 0 "R1" V 1530 8025 50  0000 C CNN
-F 1 "10kR" V 1450 8025 50  0000 C CNN
-F 2 "Resistor_SMD:R_0603_1608Metric_Pad0.98x0.95mm_HandSolder" V 1380 8025 50  0001 C CNN
-F 3 "" H 1450 8025 50  0001 C CNN
-F 4 "C25804" V 1450 8025 50  0001 C CNN "LCSC"
-	1    1450 8025
-	1    0    0    -1
-$EndComp
-Connection ~ 1450 8175
-$Comp
-L Atmega_328_breakout-rescue:R R2
-U 1 1 5A748DF6
-P 1450 8325
-F 0 "R2" V 1530 8325 50  0000 C CNN
-F 1 "20k" V 1450 8325 50  0000 C CNN
-F 2 "Resistor_SMD:R_0603_1608Metric_Pad0.98x0.95mm_HandSolder" V 1380 8325 50  0001 C CNN
-F 3 "" H 1450 8325 50  0001 C CNN
-F 4 "C4184" V 1450 8325 50  0001 C CNN "LCSC"
-	1    1450 8325
-	1    0    0    -1
-$EndComp
-$Comp
 L Atmega_328_breakout-rescue:+5V #PWR07
 U 1 1 5A748A91
@@
 F 3 "" H 1700 8375 50  0001 C CNN
 	1    1700 8375
-	1    0    0    -1
-$EndComp
-$Comp
-L Amplifier_Operational:TL071 U3
-U 1 1 5A74871A
-P 2150 8275
-F 0 "U3" H 2150 8525 50  0000 L CNN
-F 1 "TL071" H 2150 8425 50  0000 L CNN
-F 2 "Package_SO:SOIC-8_3.9x4.9mm_P1.27mm" H 2200 8325 50  0001 C CNN
-F 3 "" H 2300 8425 50  0001 C CNN
-F 4 "C350565" H 2150 8275 50  0001 C CNN "LCSC"
-	1    2150 8275
 	1    0    0    -1
 $EndComp
@@
 Wire Wire Line
 	14725 2250 15200 2250
-Text GLabel 4200 1200 2    60   BiDi ~ 0
+Text GLabel 4100 1200 2    60   BiDi ~ 0
 XTAL1(PB6)
 Wire Wire Line
 	3650 1650 3650 1850
 Wire Wire Line
-	4150 1850 4150 1650
-Wire Wire Line
-	4150 1450 4150 1200
-Wire Wire Line
-	4150 1200 4000 1200
+	4050 1850 4050 1650
 Wire Wire Line
 	3700 1200 3650 1200
 Wire Wire Line
 	3650 1200 3650 1450
-Connection ~ 4150 1200
 Wire Wire Line
 	3550 1200 3650 1200
@@
 Wire Wire Line
 	10750 2000 10750 2050
-Text GLabel 2700 8575 0    60   Input ~ 0
-VUSB
-$Comp
-L Atmega_328_breakout-rescue:+5V #PWR012
-U 1 1 5A74AA13
-P 3525 8575
-F 0 "#PWR012" H 3525 8425 50  0001 C CNN
-F 1 "+5V" H 3525 8715 50  0000 C CNN
-F 2 "" H 3525 8575 50  0001 C CNN
-F 3 "" H 3525 8575 50  0001 C CNN
-	1    3525 8575
-	1    0    0    -1
-$EndComp
-Wire Wire Line
-	3525 8575 3300 8575
-$Comp
-L Atmega_328_breakout-rescue:Q_PMOS_SGD Q1
-U 1 1 5A74A028
-P 3100 8475
-F 0 "Q1" H 3300 8525 50  0000 L CNN
-F 1 "PMOS" H 3300 8425 50  0000 L CNN
-F 2 "Package_TO_SOT_SMD:SOT-23" H 3300 8575 50  0001 C CNN
-F 3 "" H 3100 8475 50  0001 C CNN
-	1    3100 8475
-	0    1    1    0
-$EndComp
-Wire Wire Line
-	2700 8575 2900 8575
 Text GLabel 14250 8200 0    60   Input ~ 0
 VUSB
@@
 L power:GND #PWR034
 U 1 1 6000723C
-P 3900 1850
-F 0 "#PWR034" H 3900 1600 50  0001 C CNN
-F 1 "GND" H 3905 1677 50  0000 C CNN
-F 2 "" H 3900 1850 50  0001 C CNN
-F 3 "" H 3900 1850 50  0001 C CNN
-	1    3900 1850
+P 3850 1850
+F 0 "#PWR034" H 3850 1600 50  0001 C CNN
+F 1 "GND" H 3855 1677 50  0000 C CNN
+F 2 "" H 3850 1850 50  0001 C CNN
+F 3 "" H 3850 1850 50  0001 C CNN
+	1    3850 1850
 	1    0    0    -1
 $EndComp
 Wire Wire Line
 	3650 1850 3850 1850
-Connection ~ 3900 1850
-Wire Wire Line
-	3900 1850 4150 1850
 $Comp
 L power:GND #PWR045
@@
 	3850 1400 3850 1850
 Connection ~ 3850 1850
-Wire Wire Line
-	3850 1850 3900 1850
-Wire Wire Line
-	4200 1200 4150 1200
 $Comp
 L power:GND #PWR048
@@
 Wire Wire Line
 	3850 800  3850 1000
+Wire Wire Line
+	3850 1850 4050 1850
+Wire Wire Line
+	4000 1200 4050 1200
+Wire Wire Line
+	4050 1450 4050 1200
+Connection ~ 4050 1200
+Wire Wire Line
+	4050 1200 4100 1200
+$Comp
+L Atmega_328_breakout-rescue:R R2
+U 1 1 5A748DF6
+P 1450 8325
+F 0 "R2" V 1530 8325 50  0000 C CNN
+F 1 "30k" V 1450 8325 50  0000 C CNN
+F 2 "Resistor_SMD:R_0603_1608Metric_Pad0.98x0.95mm_HandSolder" V 1380 8325 50  0001 C CNN
+F 3 "" H 1450 8325 50  0001 C CNN
+F 4 "C4184" V 1450 8325 50  0001 C CNN "LCSC"
+	1    1450 8325
+	1    0    0    -1
+$EndComp
+$Comp
+L power:GND #PWR06
+U 1 1 5A7493FE
+P 1450 8475
+F 0 "#PWR06" H 1450 8225 50  0001 C CNN
+F 1 "GND" H 1450 8325 50  0000 C CNN
+F 2 "" H 1450 8475 50  0001 C CNN
+F 3 "" H 1450 8475 50  0001 C CNN
+	1    1450 8475
+	1    0    0    -1
+$EndComp
+Wire Wire Line
+	1850 8175 1450 8175
+Connection ~ 1450 8175
+Wire Wire Line
+	1450 7800 1450 7875
+Wire Wire Line
+	3100 8275 2450 8275
+Wire Wire Line
+	2700 8575 2900 8575
+$Comp
+L Atmega_328_breakout-rescue:Q_PMOS_SGD Q1
+U 1 1 5A74A028
+P 3100 8475
+F 0 "Q1" H 3300 8525 50  0000 L CNN
+F 1 "PMOS" H 3300 8425 50  0000 L CNN
+F 2 "Package_TO_SOT_SMD:SOT-23" H 3300 8575 50  0001 C CNN
+F 3 "" H 3100 8475 50  0001 C CNN
+	1    3100 8475
+	0    1    1    0
+$EndComp
+Wire Wire Line
+	3525 8575 3300 8575
+$Comp
+L Atmega_328_breakout-rescue:+5V #PWR012
+U 1 1 5A74AA13
+P 3525 8575
+F 0 "#PWR012" H 3525 8425 50  0001 C CNN
+F 1 "+5V" H 3525 8715 50  0000 C CNN
+F 2 "" H 3525 8575 50  0001 C CNN
+F 3 "" H 3525 8575 50  0001 C CNN
+	1    3525 8575
+	1    0    0    -1
+$EndComp
+Text GLabel 2700 8575 0    60   Input ~ 0
+VUSB
+NoConn ~ 2250 8575
+NoConn ~ 2150 8575
+$Comp
+L Amplifier_Operational:TL071 U3
+U 1 1 5A74871A
+P 2150 8275
+F 0 "U3" H 2150 8525 50  0000 L CNN
+F 1 "TL071" H 2150 8425 50  0000 L CNN
+F 2 "Package_SO:SOIC-8_3.9x4.9mm_P1.27mm" H 2200 8325 50  0001 C CNN
+F 3 "" H 2300 8425 50  0001 C CNN
+F 4 "C350565" H 2150 8275 50  0001 C CNN "LCSC"
+	1    2150 8275
+	1    0    0    -1
+$EndComp
+$Comp
+L Atmega_328_breakout-rescue:R R1
+U 1 1 5A749034
+P 1450 8025
+F 0 "R1" V 1530 8025 50  0000 C CNN
+F 1 "5k" V 1450 8025 50  0000 C CNN
+F 2 "Resistor_SMD:R_0603_1608Metric_Pad0.98x0.95mm_HandSolder" V 1380 8025 50  0001 C CNN
+F 3 "" H 1450 8025 50  0001 C CNN
+F 4 "C25804" V 1450 8025 50  0001 C CNN "LCSC"
+	1    1450 8025
+	1    0    0    -1
+$EndComp
 $EndSCHEMATC

Commit message: Every thing is placed and files are created.
Parts:
- added LOGO1: Logo_Open_Hardware_Large, jorgen:BB2QR, symbol Graphic:Logo_Open_Hardware_Large
- added unit 2 of U3
- added unit 3 of U3
- D3: value LED -> LED on; LCSC C188728 -> C2296
- D4: value LED -> LED user; LCSC C188728 -> C2293
- R1: value 5k -> 10k
- R2: value 30k -> 10k; LCSC C4184 -> C25804
- U3: value TL071 -> LM358; symbol Amplifier_Operational:TL071 -> Amplifier_Operational:LM358; LCSC C350565 -> C7950
Connections:
- net +5V: now also U3.8 (V+); no longer U3.7 (V+)
- net GND: now also U3.4 (V-); no longer U3.4 (V-)
- net PD0(RX): now also J26.10 (Pin_10), U6.6 (TX); no longer J26.9 (Pin_9), U6.5 (RX)
- net PD1(TX): now also J26.9 (Pin_9), U6.5 (RX); no longer J26.10 (Pin_10), U6.6 (TX)
- net at U3.1: now also U3.5 (+)
- net at Q1.2 (G): now also U3.6 (-), U3.7; no longer U3.6
- no-connect marks 11 -> 9
Other:
- moved on the sheet: Q1, R1, R2
Changed lines of the file:
@@
 P 13900 6350
 F 0 "D4" H 13900 6450 50  0000 C CNN
-F 1 "LED" H 13900 6250 50  0000 C CNN
+F 1 "LED user" H 13900 6250 50  0000 C CNN
 F 2 "LED_SMD:LED_0805_2012Metric_Pad1.15x1.40mm_HandSolder" H 13900 6350 50  0001 C CNN
 F 3 "" H 13900 6350 50  0001 C CNN
-F 4 "C188728" H 13900 6350 50  0001 C CNN "LCSC"
+F 4 "C2293" H 13900 6350 50  0001 C CNN "LCSC"
 	1    13900 6350
 	0    -1   -1   0
@@
 Text GLabel 1800 5350 0    60   BiDi ~ 0
 AGND
-Wire Wire Line
-	1700 8375 1850 8375
 NoConn ~ 1000 6650
 $Comp
@@
 L Atmega_328_breakout-rescue:+5V #PWR08
 U 1 1 5A749A57
-P 2050 7975
-F 0 "#PWR08" H 2050 7825 50  0001 C CNN
-F 1 "+5V" H 2050 8115 50  0000 C CNN
-F 2 "" H 2050 7975 50  0001 C CNN
-F 3 "" H 2050 7975 50  0001 C CNN
-	1    2050 7975
+P 3900 8150
+F 0 "#PWR08" H 3900 8000 50  0001 C CNN
+F 1 "+5V" H 3900 8290 50  0000 C CNN
+F 2 "" H 3900 8150 50  0001 C CNN
+F 3 "" H 3900 8150 50  0001 C CNN
+	1    3900 8150
 	1    0    0    -1
 $EndComp
@@
 L power:GND #PWR09
 U 1 1 5A7499E0
-P 2050 8575
-F 0 "#PWR09" H 2050 8325 50  0001 C CNN
-F 1 "GND" H 2050 8425 50  0000 C CNN
-F 2 "" H 2050 8575 50  0001 C CNN
-F 3 "" H 2050 8575 50  0001 C CNN
-	1    2050 8575
-	1    0    0    -1
-$EndComp
-$Comp
-L Atmega_328_breakout-rescue:+5V #PWR07
-U 1 1 5A748A91
-P 1700 8375
-F 0 "#PWR07" H 1700 8225 50  0001 C CNN
-F 1 "+5V" H 1700 8515 50  0000 C CNN
-F 2 "" H 1700 8375 50  0001 C CNN
-F 3 "" H 1700 8375 50  0001 C CNN
-	1    1700 8375
+P 3900 9000
+F 0 "#PWR09" H 3900 8750 50  0001 C CNN
+F 1 "GND" H 3900 8850 50  0000 C CNN
+F 2 "" H 3900 9000 50  0001 C CNN
+F 3 "" H 3900 9000 50  0001 C CNN
+	1    3900 9000
 	1    0    0    -1
 $EndComp
@@
 Wire Wire Line
 	8650 9750 9125 9750
+Text GLabel 14950 1300 2    60   BiDi ~ 0
+PD0(RX)
 Text GLabel 14100 1300 0    60   BiDi ~ 0
-PD0(RX)
-Text GLabel 14950 1300 2    60   BiDi ~ 0
 PD1(TX)
 Text GLabel 14950 1200 2    60   BiDi ~ 0
@@
 P 5100 10200
 F 0 "D3" H 5100 10300 50  0000 C CNN
-F 1 "LED" H 5100 10100 50  0000 C CNN
+F 1 "LED on" H 5100 10100 50  0000 C CNN
 F 2 "LED_SMD:LED_0805_2012Metric_Pad1.15x1.40mm_HandSolder" H 5100 10200 50  0001 C CNN
 F 3 "" H 5100 10200 50  0001 C CNN
-F 4 "C188728" H 5100 10200 50  0001 C CNN "LCSC"
+F 4 "C2296" H 5100 10200 50  0001 C CNN "LCSC"
 	1    5100 10200
 	0    -1   -1   0
@@
 NoConn ~ 13600 9100
 NoConn ~ 13600 9000
+Text GLabel 12700 9100 0    60   BiDi ~ 0
+PD0(RX)
 Text GLabel 12700 9000 0    60   BiDi ~ 0
-PD0(RX)
-Text GLabel 12700 9100 0    60   BiDi ~ 0
 PD1(TX)
 Wire Wire Line
@@
 Wire Wire Line
 	4050 1200 4100 1200
+Text GLabel 2750 9000 0    60   Input ~ 0
+VUSB
+$Comp
+L Atmega_328_breakout-rescue:+5V #PWR012
+U 1 1 5A74AA13
+P 3550 9000
+F 0 "#PWR012" H 3550 8850 50  0001 C CNN
+F 1 "+5V" H 3550 9140 50  0000 C CNN
+F 2 "" H 3550 9000 50  0001 C CNN
+F 3 "" H 3550 9000 50  0001 C CNN
+	1    3550 9000
+	1    0    0    -1
+$EndComp
+$Comp
+L Atmega_328_breakout-rescue:Q_PMOS_SGD Q1
+U 1 1 5A74A028
+P 3150 8900
+F 0 "Q1" H 3350 8950 50  0000 L CNN
+F 1 "PMOS" H 3350 8850 50  0000 L CNN
+F 2 "Package_TO_SOT_SMD:SOT-23" H 3350 9000 50  0001 C CNN
+F 3 "" H 3150 8900 50  0001 C CNN
+	1    3150 8900
+	0    1    1    0
+$EndComp
+$Comp
+L Amplifier_Operational:LM358 U3
+U 2 1 5FA0E181
+P 2850 8450
+F 0 "U3" H 2850 8700 50  0000 L CNN
+F 1 "LM358" H 2850 8600 50  0000 L CNN
+F 2 "Package_SO:SOIC-8_3.9x4.9mm_P1.27mm" H 2900 8500 50  0001 C CNN
+F 3 "" H 3000 8600 50  0001 C CNN
+F 4 "C7950" H 2850 8450 50  0001 C CNN "LCSC"
+	2    2850 8450
+	1    0    0    -1
+$EndComp
+$Comp
+L Amplifier_Operational:LM358 U3
+U 1 1 5A74871A
+P 2200 8350
+F 0 "U3" H 2200 8600 50  0000 L CNN
+F 1 "LM358" H 2200 8500 50  0000 L CNN
+F 2 "Package_SO:SOIC-8_3.9x4.9mm_P1.27mm" H 2250 8400 50  0001 C CNN
+F 3 "" H 2350 8500 50  0001 C CNN
+F 4 "C7950" H 2200 8350 50  0001 C CNN "LCSC"
+	1    2200 8350
+	1    0    0    -1
+$EndComp
+$Comp
+L Atmega_328_breakout-rescue:R R1
+U 1 1 5A749034
+P 1450 8000
+F 0 "R1" V 1530 8000 50  0000 C CNN
+F 1 "10k" V 1450 8025 50  0000 C CNN
+F 2 "Resistor_SMD:R_0603_1608Metric_Pad0.98x0.95mm_HandSolder" V 1380 8000 50  0001 C CNN
+F 3 "" H 1450 8000 50  0001 C CNN
+F 4 "C25804" V 1450 8000 50  0001 C CNN "LCSC"
+	1    1450 8000
+	1    0    0    -1
+$EndComp
+Wire Wire Line
+	1450 8300 1450 8250
+Wire Wire Line
+	1450 7850 1450 7800
+$Comp
+L power:GND #PWR06
+U 1 1 5A7493FE
+P 1450 8750
+F 0 "#PWR06" H 1450 8500 50  0001 C CNN
+F 1 "GND" H 1450 8600 50  0000 C CNN
+F 2 "" H 1450 8750 50  0001 C CNN
+F 3 "" H 1450 8750 50  0001 C CNN
+	1    1450 8750
+	1    0    0    -1
+$EndComp
+Wire Wire Line
+	1450 8750 1450 8600
+$Comp
+L Atmega_328_breakout-rescue:+5V #PWR07
+U 1 1 5A748A91
+P 1750 8450
+F 0 "#PWR07" H 1750 8300 50  0001 C CNN
+F 1 "+5V" H 1750 8590 50  0000 C CNN
+F 2 "" H 1750 8450 50  0001 C CNN
+F 3 "" H 1750 8450 50  0001 C CNN
+	1    1750 8450
+	1    0    0    -1
+$EndComp
+Wire Wire Line
+	1900 8450 1750 8450
+Wire Wire Line
+	1900 8250 1450 8250
+Connection ~ 1450 8250
+Wire Wire Line
+	1450 8250 1450 8150
+Wire Wire Line
+	2550 8350 2500 8350
+Wire Wire Line
+	3150 8450 3150 8700
+Wire Wire Line
+	3150 8700 2550 8700
+Wire Wire Line
+	2550 8700 2550 8550
+Connection ~ 3150 8700
+Wire Wire Line
+	2750 9000 2950 9000
+Wire Wire Line
+	3350 9000 3550 9000
+$Comp
+L Amplifier_Operational:LM358 U3
+U 3 1 5FEC15EB
+P 4000 8650
+F 0 "U3" H 4000 8900 50  0000 L CNN
+F 1 "LM358" H 4000 8800 50  0000 L CNN
+F 2 "Package_SO:SOIC-8_3.9x4.9mm_P1.27mm" H 4050 8700 50  0001 C CNN
+F 3 "" H 4150 8800 50  0001 C CNN
+F 4 "C7950" H 4000 8650 50  0001 C CNN "LCSC"
+	3    4000 8650
+	1    0    0    -1
+$EndComp
+Wire Wire Line
+	3900 9000 3900 8950
+Wire Wire Line
+	3900 8150 3900 8350
 $Comp
 L Atmega_328_breakout-rescue:R R2
 U 1 1 5A748DF6
-P 1450 8325
-F 0 "R2" V 1530 8325 50  0000 C CNN
-F 1 "30k" V 1450 8325 50  0000 C CNN
-F 2 "Resistor_SMD:R_0603_1608Metric_Pad0.98x0.95mm_HandSolder" V 1380 8325 50  0001 C CNN
-F 3 "" H 1450 8325 50  0001 C CNN
-F 4 "C4184" V 1450 8325 50  0001 C CNN "LCSC"
-	1    1450 8325
-	1    0    0    -1
-$EndComp
-$Comp
-L power:GND #PWR06
-U 1 1 5A7493FE
-P 1450 8475
-F 0 "#PWR06" H 1450 8225 50  0001 C CNN
-F 1 "GND" H 1450 8325 50  0000 C CNN
-F 2 "" H 1450 8475 50  0001 C CNN
-F 3 "" H 1450 8475 50  0001 C CNN
-	1    1450 8475
-	1    0    0    -1
-$EndComp
-Wire Wire Line
-	1850 8175 1450 8175
-Connection ~ 1450 8175
-Wire Wire Line
-	1450 7800 1450 7875
-Wire Wire Line
-	3100 8275 2450 8275
-Wire Wire Line
-	2700 8575 2900 8575
-$Comp
-L Atmega_328_breakout-rescue:Q_PMOS_SGD Q1
-U 1 1 5A74A028
-P 3100 8475
-F 0 "Q1" H 3300 8525 50  0000 L CNN
-F 1 "PMOS" H 3300 8425 50  0000 L CNN
-F 2 "Package_TO_SOT_SMD:SOT-23" H 3300 8575 50  0001 C CNN
-F 3 "" H 3100 8475 50  0001 C CNN
-	1    3100 8475
-	0    1    1    0
-$EndComp
-Wire Wire Line
-	3525 8575 3300 8575
-$Comp
-L Atmega_328_breakout-rescue:+5V #PWR012
-U 1 1 5A74AA13
-P 3525 8575
-F 0 "#PWR012" H 3525 8425 50  0001 C CNN
-F 1 "+5V" H 3525 8715 50  0000 C CNN
-F 2 "" H 3525 8575 50  0001 C CNN
-F 3 "" H 3525 8575 50  0001 C CNN
-	1    3525 8575
-	1    0    0    -1
-$EndComp
-Text GLabel 2700 8575 0    60   Input ~ 0
-VUSB
-NoConn ~ 2250 8575
-NoConn ~ 2150 8575
-$Comp
-L Amplifier_Operational:TL071 U3
-U 1 1 5A74871A
-P 2150 8275
-F 0 "U3" H 2150 8525 50  0000 L CNN
-F 1 "TL071" H 2150 8425 50  0000 L CNN
-F 2 "Package_SO:SOIC-8_3.9x4.9mm_P1.27mm" H 2200 8325 50  0001 C CNN
-F 3 "" H 2300 8425 50  0001 C CNN
-F 4 "C350565" H 2150 8275 50  0001 C CNN "LCSC"
-	1    2150 8275
-	1    0    0    -1
-$EndComp
-$Comp
-L Atmega_328_breakout-rescue:R R1
-U 1 1 5A749034
-P 1450 8025
-F 0 "R1" V 1530 8025 50  0000 C CNN
-F 1 "5k" V 1450 8025 50  0000 C CNN
-F 2 "Resistor_SMD:R_0603_1608Metric_Pad0.98x0.95mm_HandSolder" V 1380 8025 50  0001 C CNN
-F 3 "" H 1450 8025 50  0001 C CNN
-F 4 "C25804" V 1450 8025 50  0001 C CNN "LCSC"
-	1    1450 8025
-	1    0    0    -1
-$EndComp
+P 1450 8450
+F 0 "R2" V 1530 8450 50  0000 C CNN
+F 1 "10k" V 1450 8450 50  0000 C CNN
+F 2 "Resistor_SMD:R_0603_1608Metric_Pad0.98x0.95mm_HandSolder" V 1380 8450 50  0001 C CNN
+F 3 "" H 1450 8450 50  0001 C CNN
+F 4 "C25804" V 1450 8450 50  0001 C CNN "LCSC"
+	1    1450 8450
+	1    0    0    -1
+$EndComp
+$Comp
+L Graphic:Logo_Open_Hardware_Large LOGO1
+U 1 1 600B34C4
+P 7150 10650
+F 0 "LOGO1" H 7150 11150 50  0001 C CNN
+F 1 "Logo_Open_Hardware_Large" H 7150 10250 50  0001 C CNN
+F 2 "jorgen:BB2QR" H 7150 10650 50  0001 C CNN
+F 3 "~" H 7150 10650 50  0001 C CNN
+	1    7150 10650
+	1    0    0    -1
+$EndComp

Commit message: updated scheme
Parts:
- removed Q1: PMOS, Package_TO_SOT_SMD:SOT-23, symbol Atmega_328_breakout-rescue:Q_PMOS_SGD
- added Q1: AO3401A, Package_TO_SOT_SMD:SOT-23, symbol Transistor_FET:AO3401A
Connections:
- net +5V: now also Q1.3 (D)
- net VUSB: now also Q1.2 (S)
- net at U3.6 (-), U3.7: now also Q1.1 (G)
Changed lines of the file:
@@
 L Atmega_328_breakout-rescue:GND #PWR051
 U 1 1 61158164
-P 850 1500
-F 0 "#PWR051" H 850 1250 50  0001 C CNN
-F 1 "GND" H 850 1350 50  0000 C CNN
-F 2 "" H 850 1500 50  0001 C CNN
-F 3 "" H 850 1500 50  0001 C CNN
-	1    850  1500
+P 750 1800
+F 0 "#PWR051" H 750 1550 50  0001 C CNN
+F 1 "GND" H 750 1650 50  0000 C CNN
+F 2 "" H 750 1800 50  0001 C CNN
+F 3 "" H 750 1800 50  0001 C CNN
+	1    750  1800
 	1    0    0    -1
 $EndComp
@@
 L power:PWR_FLAG #FLG04
 U 1 1 613B8BE6
-P 1600 1500
-F 0 "#FLG04" H 1600 1575 50  0001 C CNN
-F 1 "PWR_FLAG" H 1600 1673 50  0000 C CNN
-F 2 "" H 1600 1500 50  0001 C CNN
-F 3 "~" H 1600 1500 50  0001 C CNN
-	1    1600 1500
+P 1100 1800
+F 0 "#FLG04" H 1100 1875 50  0001 C CNN
+F 1 "PWR_FLAG" H 1100 1973 50  0000 C CNN
+F 2 "" H 1100 1800 50  0001 C CNN
+F 3 "~" H 1100 1800 50  0001 C CNN
+	1    1100 1800
 	-1   0    0    1
 $EndComp
@@
 L power:VCC #PWR049
 U 1 1 613D81E8
-P 1600 1500
-F 0 "#PWR049" H 1600 1350 50  0001 C CNN
-F 1 "VCC" H 1615 1673 50  0000 C CNN
-F 2 "" H 1600 1500 50  0001 C CNN
-F 3 "" H 1600 1500 50  0001 C CNN
-	1    1600 1500
+P 1100 1800
+F 0 "#PWR049" H 1100 1650 50  0001 C CNN
+F 1 "VCC" H 1115 1973 50  0000 C CNN
+F 2 "" H 1100 1800 50  0001 C CNN
+F 3 "" H 1100 1800 50  0001 C CNN
+	1    1100 1800
 	1    0    0    -1
 $EndComp
@@
 L power:PWR_FLAG #FLG01
 U 1 1 61177CA5
-P 850 1500
-F 0 "#FLG01" H 850 1575 50  0001 C CNN
-F 1 "PWR_FLAG" H 850 1673 50  0000 C CNN
-F 2 "" H 850 1500 50  0001 C CNN
-F 3 "~" H 850 1500 50  0001 C CNN
-	1    850  1500
-	1    0    0    -1
-$EndComp
-Wire Wire Line
-	1150 2050 1250 2050
-Text GLabel 1150 2050 0    60   BiDi ~ 0
+P 750 1800
+F 0 "#FLG01" H 750 1875 50  0001 C CNN
+F 1 "PWR_FLAG" H 750 1973 50  0000 C CNN
+F 2 "" H 750 1800 50  0001 C CNN
+F 3 "~" H 750 1800 50  0001 C CNN
+	1    750  1800
+	1    0    0    -1
+$EndComp
+Text GLabel 1150 1300 2    60   BiDi ~ 0
 AGND
 $Comp
 L power:PWR_FLAG #FLG0104
 U 1 1 5F90D195
-P 1250 2050
-F 0 "#FLG0104" H 1250 2125 50  0001 C CNN
-F 1 "PWR_FLAG" H 1250 2223 50  0000 C CNN
-F 2 "" H 1250 2050 50  0001 C CNN
-F 3 "~" H 1250 2050 50  0001 C CNN
-	1    1250 2050
-	1    0    0    -1
+P 1150 1300
+F 0 "#FLG0104" H 1150 1375 50  0001 C CNN
+F 1 "PWR_FLAG" V 1150 1600 50  0000 C CNN
+F 2 "" H 1150 1300 50  0001 C CNN
+F 3 "~" H 1150 1300 50  0001 C CNN
+	1    1150 1300
+	0    -1   -1   0
 $EndComp
 Wire Wire Line
@@
 $EndComp
 $Comp
-L Atmega_328_breakout-rescue:Q_PMOS_SGD Q1
-U 1 1 5A74A028
-P 3150 8900
-F 0 "Q1" H 3350 8950 50  0000 L CNN
-F 1 "PMOS" H 3350 8850 50  0000 L CNN
-F 2 "Package_TO_SOT_SMD:SOT-23" H 3350 9000 50  0001 C CNN
-F 3 "" H 3150 8900 50  0001 C CNN
-	1    3150 8900
-	0    1    1    0
-$EndComp
-$Comp
 L Amplifier_Operational:LM358 U3
 U 2 1 5FA0E181
@@
 	1    0    0    -1
 $EndComp
+$Comp
+L Transistor_FET:AO3401A Q1
+U 1 1 5F9FD044
+P 3150 8900
+F 0 "Q1" V 3399 8900 50  0000 C CNN
+F 1 "AO3401A" V 3490 8900 50  0000 C CNN
+F 2 "Package_TO_SOT_SMD:SOT-23" H 3350 8825 50  0001 L CIN
+F 3 "http://www.aosmd.com/pdfs/datasheet/AO3401A.pdf" H 3150 8900 50  0001 L CNN
+F 4 "C15127" V 3150 8900 50  0001 C CNN "LCSC"
+	1    3150 8900
+	0    1    1    0
+$EndComp
 $EndSCHEMATC

Commit message: Initial push
Parts:
- removed U6: MCP2221, Package_SO:TSSOP-14_4.4x5mm_P0.65mm, symbol Atmega_328_breakout-rescue:MCP2221
- added C15, C16: 100n, Capacitor_SMD:C_0402_1005Metric, symbol Atmega_328_breakout-rescue:C_Small
- added R10, R13: 120, Resistor_SMD:R_0402_1005Metric, symbol Atmega_328_breakout-rescue:R
- added U6: CH340E, Package_SO:MSOP-10_3x3mm_P0.5mm, symbol Interface_USB:CH340E
Connections:
- net GND: now also C15.1, C16.1, U6.3 (GND)
- net PD0(RX): now also R10.2
- net PD1(TX): now also R13.2
- net VCC: now also C15.2, U6.7 (VCC)
- net ~RESET: now also U6.4 (~RTS)
- net at J28.2 (D-): now also U6.2 (UD-)
- net at J28.3 (D+): now also U6.1 (UD+)
- new net: C16.2, U6.10 (V3)
- new net: R10.1, U6.8 (TXD)
- new net: R13.1, U6.9 (RXD)
- no-connect marks 9 -> 5
Other:
- moved on the sheet: C14, C9, J28, R6, R7, SW1
