File: Kicad/_autosave-Atmega_328_breakout.kicad_pcb (KiCad board)
At the start: 2 copper layers, 73.8 x 62 mm, 70 parts, among them J1 Jack-DC, J10 Conn_01x06, J11 01x03, J12 01x03, J13 01x03, J14 01x03, J15 01x03, J16 01x03, J17 01x03, J18 01x03, J19 Power_connector, J2 01x03, J20 ADC_Connector, J21 PORB++_connector, J22 PORD_connector, J23 Conn_01x01, J24 Device_Connector, J25 Pin out, J26 Com_header, J27 Power terminal, J28 USB, J3 01x03, J4 01x03, J5 01x03, J6 01x03, J7 01x03, J8 01x03, J9 01x03, Q1 PMOS, SW1 SW_Push, SW2 SW_Push, U1 NCP1117-5, U2 L7805, U3 TL071, U4 ATMEGA328P-AU, U5 MCP1700-33, U6 MCP2221, Y1 Crystal_GND24

Commit message: before switching
Parts:
- moved R1 4.66 mm to (62.2, 90.5)
- moved R2 1.80 mm to (62.2, 89.0)
Routing:
- net Net-(C2-Pad2): track 30.7 -> 26.0 mm
- net GND: track 84.6 -> 80.8 mm
- net Net-(R1-Pad2): track 7.12 -> 4.04 mm
